File: KiCad/ALU.kicad_sch (KiCad schematic)
At the start: 38 parts, among them U10 74LS245, U11 74LS86, U12 74LS283, U13 74LS283, U14 74LS86, U7 74LS173, U8 74LS08, U9 74LS02

Commit message: Updates
Parts:
- gave numbers to parts that had none: 7
