File: KiCad/Control_Logic.kicad_sch (KiCad schematic)
At the start: 82 parts, among them SW8 RESET, U100 74LS00, U47 74LS00, U48 74LS161, U49 74LS138, U50 28C16, U51 28C16, U52 74LS04, U53 74LS04

Commit message: Updates
Parts:
- gave numbers to parts that had none: 6
