File: KiCad/InstructionRegister.kicad_sch (KiCad schematic)
At the start: 22 parts, among them U35 74LS245, U36 74LS173, U37 74LS173

Commit message: Updates
Parts:
- gave numbers to parts that had none: 3
