File: KiCad/Output.kicad_sch (KiCad schematic)
At the start: 28 parts, among them SW1 SW_SPDT, U18 NE555P, U19 74LS107, U20 74LS273, U21 28C16, U22 74LS139, U23 SM420561N, U24 SM420561N, U25 SM420561N, U26 SM420561N

Commit message: Updates
Parts:
- gave numbers to parts that had none: 7
