File: KiCad/RAM.kicad_sch (KiCad schematic)
At the start: 41 parts, among them SW6 SW_Push, SW7 SW_DIP_x08, U38 74LS04, U39 74LS04, U40 74LS157, U41 74189, U42 74LS00, U43 74LS245, U44 74189, U45 74LS157, U46 74LS157

Commit message: Updates
Parts:
- gave numbers to parts that had none: 8
