File: KiCad/arduino.kicad_sch (KiCad schematic)
At the start: 15 parts, among them SW5 SW_DIP_x04, SW6 SW_Push

Commit message: Updates
Parts:
- renumbered D70 to D600, R100 to R600, R100 to R601, R100 to R602, R100 to R603, R100 to R604, R100 to R605, R100 to R606, R100 to R607, R100 to R608, R100 to R609, SW5 to SW10, SW6 to SW11, SW6 to SW12
